Commit message: Cambiar lidar del JetAuto: RPLIDAR A1 -> Orbbec MS200
- nano_bridge: anade el driver oradar_lidar (MS200, dToF, 360 grados, min 0.03 m) con su SDK.
- nano_bringup.launch.py: reemplaza rplidar_node por oradar_scan (MS200 en /dev/ttyACM0,
  topic /scan, frame lidar_frame, 15 Hz, 360 grados, range 0.03-12).
- jetauto_description (lidar_a1.urdf.xacro): lidar_frame rpy 180->0 grados. El A1 tenia su 0
  hacia atras (usaba rpy=PI); el MS200 lo tiene al frente, asi que ese 180 dejaba el scan
  volteado (objeto al frente caia atras). Corrige la orientacion del scan.

File: jetauto_ros2_ws/src/jetauto_description/urdf/lidar_a1.urdf.xacro (robot description, xacro)
@@ -6,5 +6,9 @@
     name="lidar_frame_joint"
     type="fixed">
-    <origin xyz="0 0 0" rpy="0 0 ${M_PI}" />
+    <!-- MS200 (2026-06-04): rpy yaw = 0. Su 0deg crudo apunta al FRENTE del robot, asi que NO
+         necesita giro. (El RPLIDAR A1 tenia su 0deg al reves -> usaba rpy="0 0 ${M_PI}" = 180deg;
+         con el MS200 ese 180deg dejaba el scan volteado -> objeto al frente caia en 180deg/atras.)
+         Para volver al A1: restaurar rpy="0 0 ${M_PI}". -->
+    <origin xyz="0 0 0" rpy="0 0 0" />
     <parent link="lidar_link" />
     <child link="lidar_frame" />
